File: SleepyWoof.kicad_sch (KiCad schematic)
At the start: 40 parts, among them J1 Conn_01x04, U1 TLV1704

Commit message: routing tweaks
Parts:
- R18: value 0 -> 100k; now fitted
Changed lines of the file:
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@@
 		(in_bom yes)
 		(on_board yes)
-		(dnp yes)
+		(dnp no)
 		(fields_autoplaced yes)
 		(property "Reference" "R18"
@@
 			)
 		)
-		(property "Value" "0"
+		(property "Value" "100k"
 			(at 251.46 66.675 0)
 			(effects

Commit message: ordered!
Parts:
- C1, C2, C3: footprint Capacitor_Tantalum_SMD:CP_EIA-7343-31_Kemet-D -> Capacitor_Tantalum_SMD:CP_EIA-7361-38_AVX-V; DPN 478-12572-1-ND -> 478-12518-2-ND; MPN TPSE227K016T0100V -> TCN4227M025R0100
- C4, C5, C6, C7, C8: MFR Vishay Polytech -> Murata; MPN T58MM106M6R3C0500 -> GRT188R61C106KE13D
- U1: DPN 595-TLV1704AMPWPSEP -> 296-43799-2-ND; DST Mouser -> Digi-Key
Changed lines of the file:
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@@
 			)
 		)
-		(property "Footprint" "Capacitor_Tantalum_SMD:CP_EIA-7343-31_Kemet-D"
+		(property "Footprint" "Capacitor_Tantalum_SMD:CP_EIA-7361-38_AVX-V"
 			(at 58.42 53.34 0)
 			(effects
@@
 			)
 		)
-		(property "DPN" "478-12572-1-ND"
+		(property "DPN" "478-12518-2-ND"
 			(at 58.42 53.34 0)
 			(effects
@@
 			)
 		)
-		(property "MPN" "TPSE227K016T0100V"
+		(property "MPN" "TCN4227M025R0100"
 			(at 58.42 53.34 0)
 			(effects
@@
 			)
 		)
-		(property "MFR" "Vishay Polytech"
+		(property "MFR" "Murata"
 			(at 109.22 113.03 0)
 			(effects
@@
 			)
 		)
-		(property "MPN" "T58MM106M6R3C0500"
+		(property "MPN" "GRT188R61C106KE13D"
 			(at 109.22 113.03 0)
 			(effects
@@
 			)
 		)
-		(property "DST" "Mouser"
+		(property "DST" "Digi-Key"
 			(at 82.55 58.42 0)
 			(effects
@@
 			)
 		)
-		(property "DPN" "595-TLV1704AMPWPSEP"
+		(property "DPN" "296-43799-2-ND"
 			(at 82.55 58.42 0)
 			(effects
@@
 			)
 		)
-		(property "MFR" "Vishay Polytech"
+		(property "MFR" "Murata"
 			(at 180.34 116.84 0)
 			(effects
@@
 			)
 		)
-		(property "MPN" "T58MM106M6R3C0500"
+		(property "MPN" "GRT188R61C106KE13D"
 			(at 180.34 116.84 0)
 			(effects
@@
 			)
 		)
-		(property "Footprint" "Capacitor_Tantalum_SMD:CP_EIA-7343-31_Kemet-D"
+		(property "Footprint" "Capacitor_Tantalum_SMD:CP_EIA-7361-38_AVX-V"
 			(at 68.58 53.34 0)
 			(effects
@@
 			)
 		)
-		(property "DPN" "478-12572-1-ND"
+		(property "DPN" "478-12518-2-ND"
 			(at 68.58 53.34 0)
 			(effects
@@
 			)
 		)
-		(property "MPN" "TPSE227K016T0100V"
+		(property "MPN" "TCN4227M025R0100"
 			(at 68.58 53.34 0)
 			(effects
@@
 			)
 		)
-		(property "MFR" "Vishay Polytech"
+		(property "MFR" "Murata"
 			(at 190.5 116.84 0)
 			(effects
@@
 			)
 		)
-		(property "MPN" "T58MM106M6R3C0500"
+		(property "MPN" "GRT188R61C106KE13D"
 			(at 190.5 116.84 0)
 			(effects
@@
 			)
 		)
-		(property "DST" "Mouser"
+		(property "DST" "Digi-Key"
 			(at 231.14 113.03 0)
 			(effects
@@
 			)
 		)
-		(property "DPN" "595-TLV1704AMPWPSEP"
+		(property "DPN" "296-43799-2-ND"
 			(at 231.14 113.03 0)
 			(effects
@@
 			)
 		)
-		(property "DST" "Mouser"
+		(property "DST" "Digi-Key"
 			(at 129.54 110.49 0)
 			(effects
@@
 			)
 		)
-		(property "DPN" "595-TLV1704AMPWPSEP"
+		(property "DPN" "296-43799-2-ND"
 			(at 129.54 110.49 0)
 			(effects
@@
 			)
 		)
-		(property "Footprint" "Capacitor_Tantalum_SMD:CP_EIA-7343-31_Kemet-D"
+		(property "Footprint" "Capacitor_Tantalum_SMD:CP_EIA-7361-38_AVX-V"
 			(at 48.26 53.34 0)
 			(effects
@@
 			)
 		)
-		(property "Description" "220µF Molded Tantalum Capacitors 16V 2917 (7343 Metric) 100mOhm @ 100kHz"
+		(property "Description" "220µF Molded Tantalum Capacitors 25V 2924 (7361 Metric) 100mOhm @ 100kHz"
 			(at 48.26 53.34 0)
 			(effects
@@
 			)
 		)
-		(property "DPN" "478-12572-1-ND"
+		(property "DPN" "478-12518-2-ND"
 			(at 48.26 53.34 0)
 			(effects
@@
 			)
 		)
-		(property "MPN" "TPSE227K016T0100V"
+		(property "MPN" "TCN4227M025R0100"
+			(at 48.26 53.34 0)
+			(effects
+				(font
+					(size 1.27 1.27)
+				)
+				(hide yes)
+			)
+		)
+		(property "DigiKey Part Number" ""
 			(at 48.26 53.34 0)
 			(effects
@@
 			)
 		)
+		(property "Tolerance" ""
+			(at 48.26 53.34 0)
+			(effects
+				(font
+					(size 1.27 1.27)
+				)
+			)
+		)
+		(property "Power Rating" ""
+			(at 48.26 53.34 0)
+			(effects
+				(font
+					(size 1.27 1.27)
+				)
+			)
+		)
 		(pin "1"
 		)
@@
 			)
 		)
-		(property "MFR" "Vishay Polytech"
+		(property "MFR" "Murata"
 			(at 146.05 114.3 0)
 			(effects
@@
 			)
 		)
-		(property "MPN" "T58MM106M6R3C0500"
+		(property "MPN" "GRT188R61C106KE13D"
 			(at 146.05 114.3 0)
 			(effects
@@
 			)
 		)
-		(property "DST" "Mouser"
+		(property "DST" "Digi-Key"
 			(at 204.47 110.49 0)
 			(effects
@@
 			)
 		)
-		(property "DPN" "595-TLV1704AMPWPSEP"
+		(property "DPN" "296-43799-2-ND"
 			(at 204.47 110.49 0)
 			(effects
@@
 			)
 		)
-		(property "MFR" "Vishay Polytech"
+		(property "MFR" "Murata"
 			(at 227.33 86.36 0)
 			(effects
@@
 			)
 		)
-		(property "MPN" "T58MM106M6R3C0500"
+		(property "MPN" "GRT188R61C106KE13D"
 			(at 227.33 86.36 0)
 			(effects
@@
 			)
 		)
-		(property "DST" "Mouser"
+		(property "DST" "Digi-Key"
 			(at 165.1 113.03 0)
 			(effects
@@
 			)
 		)
-		(property "DPN" "595-TLV1704AMPWPSEP"
+		(property "DPN" "296-43799-2-ND"
 			(at 165.1 113.03 0)
 			(effects
